File: CW312T-CEC1702.kicad_sch (KiCad schematic)
At the start: 0 parts

Commit message: updated pcb, schematic, production files
Other:
- sheet Active_Circuitry ports: added none; removed RST
- sheet CW312T_Connector ports: added none; removed SHUNTL
- note added: "Two nets using global labels instead of hierachical since there are multiple instances of the same net on one of the pages RST SHUNTL Double check this"
Changed lines of the file:
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@@
+		)
+	)
+	(text "Two nets using global labels instead of hierachical since there are multiple instances of the same net on one of the pages \nRST \nSHUNTL\nDouble check this "
+		(exclude_from_sim no)
+		(at 98.298 165.608 0)
+		(effects
+			(font
+				(size 1.27 1.27)
+			)
 		)
 	)
@@
 				)
 				(justify right)
-			)
-		)
-		(pin "SHUNTL" input
-			(at 92.71 148.59 270)
-			(effects
-				(font
-					(size 1.27 1.27)
-				)
-				(justify left)
 			)
 		)
@@
 			(effects
 				(font
-					(size 1.27 1.27)
-				)
-				(justify left)
-			)
-		)
-		(pin "RST" input
-			(at 205.74 149.86 270)
-			(effects
-				(font
